File: inverter_modbus/inverter_modbus.kicad_sch (KiCad schematic)
At the start: 5 parts

Commit message: Update yaml
Connections:
- net RXD: now also Brd?.13 (SDA/D2); no longer Brd?.15 (RX)
- net TXD: now also Brd?.14 (SCL/D1); no longer Brd?.16 (TX)
Changed lines of the file:
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@@
     (stroke (width 0) (type default))
   )
-  (wire (pts (xy 43.18 63.5) (xy 50.8 63.5))
+  (wire (pts (xy 71.12 55.88) (xy 78.74 55.88))
     (stroke (width 0) (type default))
   )
@@
     (stroke (width 0) (type default))
   )
+  (wire (pts (xy 71.12 58.42) (xy 78.74 58.42))
+    (stroke (width 0) (type default))
+  )
   (wire (pts (xy 101.6 86.36) (xy 107.95 86.36))
     (stroke (width 0) (type default))
@@
   )
   (wire (pts (xy 128.27 52.07) (xy 134.62 52.07))
-    (stroke (width 0) (type default))
-  )
-  (wire (pts (xy 43.18 60.96) (xy 50.8 60.96))
     (stroke (width 0) (type default))
   )
@@
     (effects (font (size 1.27 1.27)) (justify left bottom))
   )
-  (label "RXD" (at 44.45 60.96 0) (fields_autoplaced)
+  (label "RXD" (at 72.39 58.42 0) (fields_autoplaced)
     (effects (font (size 1.27 1.27)) (justify left bottom))
   )
@@
     (effects (font (size 1.27 1.27)) (justify left bottom))
   )
-  (label "TXD" (at 44.45 63.5 0) (fields_autoplaced)
-    (effects (font (size 1.27 1.27)) (justify left bottom))
-  )
+  (label "TXD" (at 72.39 55.88 0) (fields_autoplaced)
+    (effects (font (size 1.27 1.27)) (justify left bottom))
+  )
